File: 80cvc.kicad_pcb (KiCad board)
At the start: 2 copper layers, 228.6 x 139.7 mm, 78 parts, among them J1 VideoOut, J2 Conn_01x03, P1 80cvc_50_edgecard, Q1 2N3904, Q2 2N3904, U1 74LS20, U10 74LS157, U11 74LS157, U12 74LS86, U13 74LS85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

Commit message: Add files via upload
Connections:
- P1 pad 10: (no net) -> unconnected-(P1-!IRQ-Pad10)
- P1 pad 11: (no net) -> unconnected-(P1-AC-Pad11)
- P1 pad 14: (no net) -> unconnected-(P1-!ABUFFSEL-Pad14)
- P1 pad 16: (no net) -> unconnected-(P1--12V-Pad16)
- P1 pad 24: (no net) -> unconnected-(P1-+5V_REF-Pad24)
- P1 pad 26: (no net) -> unconnected-(P1-Pin_39_P1-Pad26)
- P1 pad 28: (no net) -> unconnected-(P1-Pin_39_P1-Pad28)
- P1 pad 30: (no net) -> unconnected-(P1-PIN_47_P1-Pad30)
- P1 pad 4: (no net) -> unconnected-(P1-AUDIO-Pad4)
- P1 pad 49: (no net) -> unconnected-(P1-COMPGNDRET-Pad49)
- P1 pad 5: (no net) -> unconnected-(P1-!EXTENB-Pad5)
- P1 pad 50: (no net) -> unconnected-(P1-+12V-Pad50)
- P1 pad 7: (no net) -> unconnected-(P1-!REF-Pad7)
- P1 pad 9: (no net) -> unconnected-(P1-RDY-Pad9)
- U13 pad 5: (no net) -> unconnected-(U13-Oa>b-Pad5)
- U13 pad 7: (no net) -> unconnected-(U13-Oa<b-Pad7)
- U2 pad 15: (no net) -> unconnected-(U2-MA11-Pad15)
- U2 pad 16: (no net) -> unconnected-(U2-MA12-Pad16)
- U2 pad 17: (no net) -> unconnected-(U2-MA13-Pad17)
- U2 pad 3: (no net) -> unconnected-(U2-LPSTB-Pad3)
- U2 pad 34: (no net) -> unconnected-(U2-RA4-Pad34)
- U2 pad 35: (no net) -> /R3
- U23 pad 8: (no net) -> unconnected-(U23B-~{Q}-Pad8)
- U4 pad 17: (no net) -> unconnected-(U4-I/O-Pad17)
- U6 pad 6: (no net) -> unconnected-(U6A-~{Q}-Pad6)
- U6 pad 9: (no net) -> unconnected-(U6B-Q-Pad9)
- U7 pad 11: (no net) -> unconnected-(U7-O4-Pad11)
- U7 pad 12: (no net) -> unconnected-(U7-O3-Pad12)
- U7 pad 13: (no net) -> unconnected-(U7-O2-Pad13)
- U7 pad 14: (no net) -> unconnected-(U7-O1-Pad14)
- U7 pad 15: (no net) -> unconnected-(U7-O0-Pad15)
- U7 pad 7: (no net) -> unconnected-(U7-O7-Pad7)
- U8 pad 2: (no net) -> unconnected-(U8-Q0-Pad2)
- U8 pad 3: (no net) -> unconnected-(U8-D0-Pad3)
- U9 pad 10: (no net) -> unconnected-(U9-I1c-Pad10)
- U9 pad 11: (no net) -> unconnected-(U9-I0c-Pad11)
- U9 pad 9: (no net) -> unconnected-(U9-Zc-Pad9)
Routing:
- net /DSEL: track 141.8 -> 59.6 mm, vias 1 -> 0
- net /DBUFSEL: track 0.00 -> 73.2 mm, vias 0 -> 1
- net GND: vias 114 -> 116
- net (no net): vias 4 -> 0
