File: 80cvc.kicad_sch (KiCad schematic)
At the start: 78 parts, among them J1 VideoOut, J2 Conn_01x03, P1 80cvc_50_edgecard, Q1 2N3904, Q2 2N3904, U1 74LS20, U10 74LS157, U11 74LS157, U12 74LS86, U13 74LS85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

Commit message: Add files via upload
Changed lines of the file:
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@@
   (junction (at 127 360.68) (diameter 0) (color 0 0 0 0)
   )
+  (junction (at 496.57 299.72) (diameter 0) (color 0 0 0 0)
+  )
   (junction (at 401.32 123.19) (diameter 0) (color 0 0 0 0)
   )
@@
     (stroke (width 0) (type default))
   )
+  (wire (pts (xy 471.17 289.56) (xy 471.17 298.45))
+    (stroke (width 0) (type default))
+  )
   (wire (pts (xy 157.48 350.52) (xy 157.48 353.06))
     (stroke (width 0) (type default))
@@
     (stroke (width 0) (type default))
   )
+  (wire (pts (xy 487.68 299.72) (xy 496.57 299.72))
+    (stroke (width 0) (type default))
+  )
   (wire (pts (xy 227.33 236.22) (xy 248.92 236.22))
     (stroke (width 0) (type default))
@@
     (stroke (width 0) (type default))
   )
-  (wire (pts (xy 496.57 289.56) (xy 496.57 303.53))
+  (wire (pts (xy 496.57 289.56) (xy 496.57 299.72))
     (stroke (width 0) (type default))
   )
@@
     (stroke (width 0) (type default))
   )
-  (wire (pts (xy 477.52 289.56) (xy 477.52 303.53))
-    (stroke (width 0) (type default))
-  )
   (wire (pts (xy 260.35 68.58) (xy 171.45 68.58))
     (stroke (width 0) (type default))
@@
     (stroke (width 0) (type default))
   )
+  (wire (pts (xy 471.17 298.45) (xy 461.01 298.45))
+    (stroke (width 0) (type default))
+  )
   (bus (pts (xy 72.39 184.15) (xy 72.39 186.69))
     (stroke (width 0) (type default))
@@
     (stroke (width 0) (type default))
   )
-  (wire (pts (xy 480.06 289.56) (xy 477.52 289.56))
+  (wire (pts (xy 471.17 289.56) (xy 480.06 289.56))
     (stroke (width 0) (type default))
   )
@@
     (stroke (width 0) (type default))
   )
+  (wire (pts (xy 496.57 299.72) (xy 496.57 303.53))
+    (stroke (width 0) (type default))
+  )
   (wire (pts (xy 427.99 308.61) (xy 443.23 308.61))
     (stroke (width 0) (type default))
@@
     (stroke (width 0) (type default))
   )
-  (wire (pts (xy 487.68 298.45) (xy 487.68 295.91))
+  (wire (pts (xy 487.68 295.91) (xy 487.68 299.72))
     (stroke (width 0) (type default))
   )
@@
     (stroke (width 0) (type default))
   )
-  (wire (pts (xy 461.01 298.45) (xy 487.68 298.45))
-    (stroke (width 0) (type default))
-  )
   (wire (pts (xy 157.48 360.68) (xy 162.56 360.68))
     (stroke (width 0) (type default))
@@
         )
       )
-    )
-  )
-  (symbol (lib_id "power:GND") (at 477.52 303.53 0) (unit 1)
-    (in_bom yes) (on_board yes) (dnp no)
-    (property "Reference" "#PWR0148" (at 477.52 309.88 0)
-      (effects (font (size 1.27 1.27)) hide)
-    )
-    (property "Value" "GND" (at 477.647 307.9242 0)
-      (effects (font (size 1.27 1.27)))
-    )
-    (property "Footprint" "" (at 477.52 303.53 0)
-      (effects (font (size 1.27 1.27)) hide)
-    )
-    (property "Datasheet" "" (at 477.52 303.53 0)
-      (effects (font (size 1.27 1.27)) hide)
-    )
-    (pin "1")
-    (instances
-      (project "80cvc"
-        (path "/b10f90c5-364f-4324-8c26-2a327d03a937"
-          (reference "#PWR0148") (unit 1)
-        )
-      )
